File: kitty.sch (KiCad schematic (older format))
At the start: 4 parts

Commit message: finish layout
Parts:
- SAO1: footprint Pin_Headers:Pin_Header_Angled_2x02_Pitch2.54mm -> Pin_Headers:Pin_Header_Straight_2x02_Pitch2.54mm
Changed lines of the file:
@@
 LIBS:contrib
 LIBS:valves
-LIBS:bzkhs_sheered_shenzen-cache
+LIBS:kitty-cache
 EELAYER 25 0
 EELAYER END
@@
 F 0 "SAO1" H 1350 950 50  0000 C CNN
 F 1 "2x2" H 1350 650 50  0000 C CNN
-F 2 "Pin_Headers:Pin_Header_Angled_2x02_Pitch2.54mm" H 1300 850 50  0001 C CNN
+F 2 "Pin_Headers:Pin_Header_Straight_2x02_Pitch2.54mm" H 1300 850 50  0001 C CNN
 F 3 "" H 1300 850 50  0001 C CNN
 	1    1300 850
@@
 $EndComp
 $Comp
-L +3.3V #PWR1
+L +3.3V #PWR01
 U 1 1 5B50D30A
 P 950 850
-F 0 "#PWR1" H 950 700 50  0001 C CNN
+F 0 "#PWR01" H 950 700 50  0001 C CNN
 F 1 "+3.3V" H 950 990 50  0000 C CNN
 F 2 "" H 950 850 50  0001 C CNN
@@
 	950  850  1100 850
 $Comp
-L GND #PWR2
+L GND #PWR02
 U 1 1 5B50D32A
 P 1000 1050
-F 0 "#PWR2" H 1000 800 50  0001 C CNN
+F 0 "#PWR02" H 1000 800 50  0001 C CNN
 F 1 "GND" H 1000 900 50  0000 C CNN
 F 2 "" H 1000 1050 50  0001 C CNN
@@
 $EndComp
 $Comp
-L GND #PWR3
+L GND #PWR03
 U 1 1 5B50D3A1
 P 1950 950
-F 0 "#PWR3" H 1950 700 50  0001 C CNN
+F 0 "#PWR03" H 1950 700 50  0001 C CNN
 F 1 "GND" H 1950 800 50  0000 C CNN
 F 2 "" H 1950 950 50  0001 C CNN
@@
 	1950 850  1950 950
 $Comp
-L +3.3V #PWR4
+L +3.3V #PWR04
 U 1 1 5B50D403
 P 3250 850
-F 0 "#PWR4" H 3250 700 50  0001 C CNN
+F 0 "#PWR04" H 3250 700 50  0001 C CNN
 F 1 "+3.3V" H 3250 990 50  0000 C CNN
 F 2 "" H 3250 850 50  0001 C CNN
